File: ArduinoMega2560/ArduinoMega2560.kicad_sch (KiCad schematic)
At the start: 28 parts, among them J1 Conn_02x08, J2 Conn_02x08, Q1 Crystal_16MHz, Q2 Crystal_16MHz, SW1 Push_Button, U1 ATmega2560-16A, Y1 TSX-3225_16.0000MF18X-AC0

Commit message: 1st update
Parts:
- removed C14, C15, C16, C17: 22pF_0603_16V, PCM_4ms_Capacitor:C_0603, symbol PCM_4ms_Capacitor:100nF_0603_16V
- removed Q1, Q2: Crystal_16MHz, Crystal:Crystal_HC49-4H_Vertical, symbol PCM_SL_Devices:Crystal_16MHz
Other:
- added sheet Excluded (Excluded.kicad_sch)
