File: ArduinoMega2560/ArduinoMega2560.kicad_sch (KiCad schematic)
At the start: 29 parts, among them J12 PINHD_1x6_Male, Q1 Crystal_16MHz, Q2 Crystal_16MHz, SW1 Push_Button, U1 ATmega2560-16A, Y1 TSX-3225_16.0000MF18X-AC0

Commit message: Annotation problem
Parts:
- renumbered RN1A1 to RN1A
Changed lines of the file:
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@@
   (symbol (lib_id "PCM_Resistor_AKL:R_0603") (at 87.63 58.42 180) (unit 1)
     (in_bom yes) (on_board yes) (dnp no)
-    (property "Reference" "RN1A1" (at 90.17 57.15 0)
+    (property "Reference" "RN1A" (at 90.17 57.15 0)
       (effects (font (size 1.27 1.27)) (justify right))
     )
@@
       (project "ArduinoMega2560"
         (path "/9c604cc5-1a6f-41a9-b015-ecf51c009c14"
-          (reference "RN1A1") (unit 1)
+          (reference "RN1A") (unit 1)
         )
       )

Commit message: Daily update
Parts:
- renumbered J_PWR1 to PWR1, RN1A to RN1A1

Commit message: Update label
Parts:
- renumbered J_ADCH1 to ADCH1, RN1A1 to RN11, RN1B1 to RN12, RN1C1 to RN13
Connections:
- net RESET renamed RESET1
Other:
- sheet ATmega8U2-MU ports: added RESET1; removed RESET
- moved on the sheet: C1, C14, C15, C16, C17, ICSP2, J12, PWR1, Q1, Q2, RN11, SW1

Commit message: Tracing
Parts:
- removed PWR1: PINHD_1x4_Male, Connector_PinHeader_2.54mm:PinHeader_1x04_P2.54mm_Vertical, symbol PCM_SL_Pin_Headers:PINHD_1x4_Male
- renumbered J12 to PWR1
Other:
- sheet Power ports: added PB7; removed none

Commit message: Update Trace
Parts:
- renumbered J_ADCL1 to ADC1, ADCH1 to ADC2, J_COM1 to COM1, J_XIOH1 to J1, J_XIOL1 to J2, J_PWML1 to PWM1, J_PWM1 to PWM2
Changed lines of the file:
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@@
 		(dnp no)
 		(fields_autoplaced yes)
-		(property "Reference" "J_XIOL1"
+		(property "Reference" "J2"
 			(at 317.5 95.25 0)
 			(effects
@@
 			(project "ArduinoMega2560"
 				(path "/9c604cc5-1a6f-41a9-b015-ecf51c009c14"
-					(reference "J_XIOL1")
+					(reference "J2")
 					(unit 1)
 				)
@@
 		(on_board yes)
 		(dnp no)
-		(property "Reference" "ADCH1"
+		(property "Reference" "ADC2"
 			(at 171.45 107.95 0)
 			(effects
@@
 			(project "ArduinoMega2560"
 				(path "/9c604cc5-1a6f-41a9-b015-ecf51c009c14"
-					(reference "ADCH1")
+					(reference "ADC2")
 					(unit 1)
 				)
@@
 		(dnp no)
 		(fields_autoplaced yes)
-		(property "Reference" "J_PWML1"
+		(property "Reference" "PWM1"
 			(at 273.05 153.67 0)
 			(effects
@@
 			(project "ArduinoMega2560"
 				(path "/9c604cc5-1a6f-41a9-b015-ecf51c009c14"
-					(reference "J_PWML1")
+					(reference "PWM1")
 					(unit 1)
 				)
@@
 		(dnp no)
 		(fields_autoplaced yes)
-		(property "Reference" "J_XIOH1"
+		(property "Reference" "J1"
 			(at 317.5 52.07 0)
 			(effects
@@
 			(project "ArduinoMega2560"
 				(path "/9c604cc5-1a6f-41a9-b015-ecf51c009c14"
-					(reference "J_XIOH1")
+					(reference "J1")
 					(unit 1)
 				)
@@
 		(dnp no)
 		(fields_autoplaced yes)
-		(property "Reference" "J_COM1"
+		(property "Reference" "COM1"
 			(at 323.85 147.32 0)
 			(effects
@@
 			(project "ArduinoMega2560"
 				(path "/9c604cc5-1a6f-41a9-b015-ecf51c009c14"
-					(reference "J_COM1")
+					(reference "COM1")
 					(unit 1)
 				)
@@
 		(dnp no)
 		(fields_autoplaced yes)
-		(property "Reference" "J_ADCL1"
+		(property "Reference" "ADC1"
 			(at 273.05 176.53 0)
 			(effects
@@
 			(project "ArduinoMega2560"
 				(path "/9c604cc5-1a6f-41a9-b015-ecf51c009c14"
-					(reference "J_ADCL1")
+					(reference "ADC1")
 					(unit 1)
 				)
@@
 		(dnp no)
 		(fields_autoplaced yes)
-		(property "Reference" "J_PWM1"
+		(property "Reference" "PWM2"
 			(at 273.05 90.17 0)
 			(effects
@@
 			(project "ArduinoMega2560"
 				(path "/9c604cc5-1a6f-41a9-b015-ecf51c009c14"
-					(reference "J_PWM1")
+					(reference "PWM2")
 					(unit 1)
 				)
@@
 	(sheet
 		(at 41.91 55.88)
-		(size 25.4 35.56)
+		(size 25.4 15.24)
 		(exclude_from_sim no)
 		(in_bom yes)
@@
 		)
 		(property "Sheetfile" "arduinomega_atmega8u2.kicad_sch"
-			(at 41.91 92.0246 0)
+			(at 41.91 71.7046 0)
 			(effects
 				(font

Commit message: Update trace
Other:
- moved on the sheet: C14, C15, C16, C17, Q1, Q2

Commit message: Update trace
Parts:
- removed C14, C15: 22pF_0603_16V, PCM_4ms_Capacitor:C_0603, symbol PCM_4ms_Capacitor:100nF_0603_16V
- removed Q1: Crystal_16MHz, Crystal:Crystal_HC49-4H_Vertical, symbol PCM_SL_Devices:Crystal_16MHz
- renumbered C17 to C14, C16 to C15
Connections:
- net +3V3: now also PWR1.2; no longer PWR1.3
- net +5V: now also PWR1.3; no longer PWR1.2
- net at R1.1, U1.33 (XTAL2), Y1.3: now also C15.1, Q2.1
- net at R1.2, R3.1, Y1.1: now also C14.1, Q2.2
Other:
- added sheet Excluded (Excluded.kicad_sch)
- moved on the sheet: C14, C15, Q2
