File: ArduinoMega2560/ArduinoMega2560.kicad_pcb (KiCad board)
At the start: 2 copper layers, 101.6 x 53.3 mm, 73 parts, among them J2 UJ2-BH-1-TH, Q1 Crystal_16MHz, Q2 Crystal_16MHz, SW1 Push_Button, T2 FDN340P, U1 ATmega2560-16A, U2 ATmega8U2-A, U3 LM358D, Y1 TSX-3225_16.0000MF18X-AC0, Y2 TSX-3225_16.0000MF18X-AC0

Commit message: Update tracing
Parts:
- moved C9 100.3 mm to (59.1, 131.7)
- moved RN51 99.1 mm to (56.2, 132.5), turned to -90 degrees
- moved UBOOT1 86.9 mm to (83.4, 135.6)
- moved JP_GND1 81.3 mm to (79.8, 135.6)
- moved RESET_EN1 78.8 mm to (87.0, 135.6)
- moved C7 76.7 mm to (84.2, 141.5)
- moved C10 50.4 mm to (69.0, 117.3), turned to -90 degrees
- moved ICSP2 36.3 mm to (96.7, 139.8)
- moved U1 19.1 mm to (116.9, 134.0)
- moved ICSP1 18.6 mm to (62.3, 114.5), turned to 0 degrees
- moved LED_PB7 14.1 mm to (65.5, 106.0), turned to -90 degrees
- moved C11 13.6 mm to (67.1, 122.7), turned to 180 degrees
- moved UP3 12.4 mm to (60.0, 136.5), turned to 0 degrees
- moved C12 11.6 mm to (70.2, 137.2), turned to 0 degrees
- moved ON1 11.5 mm to (62.6, 106.0), turned to -90 degrees
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- renumbered J_ADCL1 to ADC1, ADCH1 to ADC2, J_COM1 to COM1, J_XIOH1 to J1, J_XIOL1 to J2, J_PWML1 to PWM1, J_PWM1 to PWM2, J2 to USB1
Connections:
- C7 pad 2: Net-(RESET_EN1-A) -> Net-(RESET_EN1-B)
- RESET_EN1 pad 1: Net-(RESET_EN1-A) -> RESET1
- RESET_EN1 pad 2: RESET1 -> Net-(RESET_EN1-B)
Routing:
- net +5V: track 90.1 -> 139.6 mm
- net RESET2: track 0.00 -> 20.8 mm, vias 0 -> 2
- net /Power/GATE_CMD: track 8.02 -> 18.9 mm
- net +3V3: track 47.8 -> 39.7 mm, vias 1 -> 2
- net GND: track 210.4 -> 218.1 mm, vias 5 -> 4
- net Net-(U3B-+): track 9.04 -> 16.7 mm, vias 1 -> 0
- net Net-(RESET_EN1-B): track 0.00 -> 4.87 mm
- net Net-(C8-Pad1): track 19.4 -> 15.8 mm
- net Net-(U2-~{HWB}/PD7): track 0.00 -> 3.36 mm
- net VIN: track 98.7 -> 101.4 mm
- net Net-(R2-Pad2): track 7.77 -> 9.00 mm
- net Net-(D2-Pad2): track 37.5 -> 36.8 mm

Commit message: Update tracing
Parts:
- moved TX1 74.1 mm to (89.8, 124.9)
- moved RX1 73.5 mm to (89.8, 127.2)
- moved RN41 62.3 mm to (93.3, 131.8)
- moved RN44 62.2 mm to (93.3, 127.2)
- moved RN43 62.1 mm to (93.3, 124.9)
- moved RN42 61.9 mm to (93.3, 129.5)
- moved RESET_EN1 27.5 mm to (69.5, 114.4), turned to 90 degrees
- moved C7 26.8 mm to (75.4, 116.2), turned to 90 degrees
- moved UBOOT1 23.2 mm to (69.5, 117.0), turned to 90 degrees
- moved JP_GND1 19.0 mm to (69.5, 119.6), turned to 90 degrees
- moved ICSP2 9.66 mm to (87.5, 136.8), turned to -90 degrees
- moved C10 6.56 mm to (71.4, 123.4)
- moved R2 6.38 mm to (72.5, 129.6), turned to 0 degrees
- moved U2 5.39 mm to (81.5, 124.3)
- moved U1 4.61 mm to (117.2, 138.6)
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Routing:
- net TXD0: track 0.00 -> 47.9 mm
- net RXD0: track 0.00 -> 47.9 mm
- net Net-(U2-D+): track 0.00 -> 41.1 mm
- net Net-(U2-D-): track 0.00 -> 40.7 mm
- net RESET1: track 6.50 -> 30.4 mm
- net USBVCC: track 2.30 -> 24.2 mm, vias 0 -> 2
- net Net-(U2-PC0/XTAL2): track 2.21 -> 20.0 mm, vias 0 -> 2
- net +5V: track 139.6 -> 154.3 mm, vias 0 -> 1
- net Net-(JP_GND1-A): track 18.0 -> 29.9 mm, vias 1 -> 3
- net GND: track 218.1 -> 229.4 mm, vias 4 -> 11
- net +3V3: track 39.7 -> 51.0 mm, vias 2 -> 1
- net Net-(U2-PD2): track 0.00 -> 9.52 mm
- net Net-(U2-XTAL1): track 0.00 -> 9.52 mm
- net Net-(U2-PD3): track 0.00 -> 9.48 mm
- net Net-(U2-UCAP): track 0.00 -> 6.08 mm, vias 0 -> 2
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
Commit message: Update Tracing
Parts:
- moved C11 7.78 mm to (72.3, 126.4), turned to 0 degrees
Routing:
- net RESET1: track 30.4 -> 92.2 mm, vias 0 -> 2
- net +5V: track 154.3 -> 213.5 mm, vias 1 -> 4
- net /ATmega8U2-MU/SCK: track 0.00 -> 39.9 mm, vias 0 -> 1
- net /PB3: track 0.00 -> 37.9 mm
- net /ATmega8U2-MU/MOSI: track 0.00 -> 32.6 mm, vias 0 -> 1
- net /ATmega8U2-MU/MISO: track 0.00 -> 32.3 mm, vias 0 -> 1
- net RESET2: track 20.8 -> 50.7 mm, vias 2 -> 4
- net /PB1: track 0.00 -> 28.5 mm
- net /PB2: track 0.00 -> 26.9 mm
- net /PB7: track 0.00 -> 25.0 mm, vias 0 -> 1
- net Net-(U2-~{HWB}/PD7): track 3.36 -> 27.4 mm, vias 0 -> 1
- net Net-(JP_GND1-A): track 29.9 -> 37.9 mm
- net GND: track 229.4 -> 237.4 mm, vias 11 -> 10
- net /Power/GATE_CMD: track 17.7 -> 12.0 mm
- net Net-(D2-Pad1): track 25.9 -> 21.5 mm
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
Commit message: Update trace
Parts:
- moved C1 102.0 mm to (75.7, 154.0), turned to 180 degrees
- moved RN11 96.6 mm to (75.7, 151.9), turned to 180 degrees
- moved R1 66.1 mm to (109.6, 144.9), turned to -90 degrees
- moved C6 65.4 mm to (107.0, 144.9), turned to -90 degrees
- moved Y1 65.0 mm to (112.8, 145.0), turned to 90 degrees
- moved R3 63.8 mm to (112.5, 147.8)
- moved C3 50.8 mm to (110.8, 117.4), turned to 180 degrees
- moved RN13 47.4 mm to (117.8, 149.3), turned to 180 degrees
- moved RN12 47.3 mm to (117.8, 147.5), turned to 180 degrees
- moved C4 40.4 mm to (122.2, 118.8), turned to 90 degrees
- moved C5 37.3 mm to (122.2, 115.4), turned to 90 degrees
- moved U1 7.64 mm to (117.4, 131.0)
- moved ICSP2 4.73 mm to (87.9, 132.1)
Routing:
- net GND: track 237.4 -> 325.6 mm, vias 10 -> 17
- net /PB7: track 25.0 -> 98.7 mm, vias 1 -> 4
- net +5V: track 213.5 -> 279.7 mm, vias 4 -> 11
- net Net-(U1-PE5): track 0.00 -> 56.3 mm, vias 0 -> 2
- net Net-(U1-PE4): track 0.00 -> 52.9 mm
- net /PH3: track 0.00 -> 48.1 mm, vias 0 -> 2
- net Net-(U1-PE3): track 0.00 -> 45.9 mm, vias 0 -> 2
- net /PG5: track 0.00 -> 45.6 mm
- net RESET1: track 92.2 -> 137.8 mm, vias 2 -> 4
- net /PH4: track 0.00 -> 44.9 mm, vias 0 -> 2
- net /ADC0: track 0.00 -> 37.1 mm
- net /ADC1: track 0.00 -> 35.2 mm
- net /ADC2: track 0.00 -> 33.2 mm
- net /ADC3: track 0.00 -> 31.3 mm
- net /PH5: track 0.00 -> 30.2 mm, vias 0 -> 2
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
Commit message: Update trace
Parts:
- moved Q1 26.6 mm to (154.5, 117.3)
- moved Q2 14.3 mm to (154.5, 103.3)
- moved C16 13.5 mm to (152.5, 122.0)
- moved C17 13.5 mm to (152.5, 124.6)
- moved C14 5.32 mm to (152.5, 108.0)
- moved C15 5.32 mm to (152.5, 110.7)
- moved C6 4.72 mm to (102.4, 144.0)
- moved R1 4.72 mm to (105.0, 144.0)
- moved Y1 4.72 mm to (108.2, 144.1)
- moved R3 3.84 mm to (111.4, 144.1), turned to 90 degrees
- moved RN12 2.73 mm to (116.3, 149.8), turned to -90 degrees
- moved RN13 0.56 mm to (118.1, 149.8), turned to -90 degrees
Connections:
- C15 pad 1: Net-(C15-Pad1) -> Net-(U1-XTAL2)
- C16 pad 1: Net-(C16-Pad1) -> XT1
- C17 pad 1: Net-(C17-Pad1) -> XT2
- PWR1 pad 2: +5V -> +3V3
- PWR1 pad 3: +3V3 -> +5V
- Q1 pad 1: Net-(C14-Pad1) -> XT2
- Q1 pad 2: Net-(C15-Pad1) -> XT1
- Q2 pad 1: Net-(C16-Pad1) -> Net-(U1-XTAL2)
- Q2 pad 2: Net-(C17-Pad1) -> Net-(C14-Pad1)
- R1 pad 2: Net-(R1-Pad2) -> Net-(C14-Pad1)
- R2 pad 1: Net-(U2-PC0/XTAL2) -> XT2
- R2 pad 2: Net-(R2-Pad2) -> XT1
- R3 pad 1: Net-(R1-Pad2) -> Net-(C14-Pad1)
- R4 pad 1: Net-(R2-Pad2) -> XT1
- U2 pad 2: Net-(U2-PC0/XTAL2) -> XT2
- Y1 pad 1: Net-(R1-Pad2) -> Net-(C14-Pad1)
- Y2 pad 1: Net-(R2-Pad2) -> XT1
- Y2 pad 3: Net-(U2-PC0/XTAL2) -> XT2
Routing:
- net /PL1: track 0.00 -> 46.6 mm, vias 0 -> 2
- net /PL0: track 0.00 -> 38.9 mm, vias 0 -> 2
- net /PL2: track 0.00 -> 35.3 mm, vias 0 -> 2
- net /PG2: track 0.00 -> 33.9 mm, vias 0 -> 2
- net +5V: track 279.7 -> 246.5 mm, vias 11 -> 10
- net /PL4: track 0.00 -> 32.2 mm, vias 0 -> 2
- net /PL7: track 0.00 -> 30.1 mm, vias 0 -> 2
- net /PL5: track 0.00 -> 30.1 mm, vias 0 -> 2
- net /PL3: track 0.00 -> 29.9 mm, vias 0 -> 2
- net /PL6: track 0.00 -> 29.6 mm, vias 0 -> 2
- net +3V3: track 51.0 -> 22.6 mm
- net XT2: track 0.00 -> 20.5 mm, vias 0 -> 2
- net Net-(U2-PC0/XTAL2): track 20.5 -> 0.00 mm, vias 2 -> 0
- net Net-(C14-Pad1): track 0.00 -> 8.54 mm
- net GND: track 325.6 -> 332.1 mm
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
Commit message: Update
Parts:
- added J3: PINHD_1x2_Male, Connector_PinHeader_2.54mm:PinHeader_1x02_P2.54mm_Vertical, F.Cu at (154.8, 124.5)
- added J4: PINHD_1x2_Male, Connector_PinHeader_2.54mm:PinHeader_1x02_P2.54mm_Vertical, F.Cu at (159.4, 124.5)
- moved PWM2 50.3 mm to (82.2, 105.6), turned to -90 degrees
- moved COM1 49.4 mm to (126.4, 105.7), turned to -90 degrees
- moved ADC2 48.1 mm to (116.8, 153.7)
- moved ADC1 47.6 mm to (93.9, 153.5)
- moved PWM1 34.9 mm to (104.2, 105.7), turned to -90 degrees
- moved RN33 21.5 mm to (75.7, 126.7)
- moved RN34 21.5 mm to (78.6, 126.7)
- moved ON1 21.5 mm to (75.7, 123.1)
- moved LED_PB7 21.5 mm to (78.6, 123.1)
- moved C15 14.8 mm to (159.8, 97.8)
- moved C14 14.8 mm to (159.8, 95.2)
- moved C16 14.8 mm to (159.8, 109.2)
- moved C17 14.8 mm to (159.8, 111.8)
- moved Q1 14.8 mm to (161.8, 104.5)
- moved Q2 14.8 mm to (161.8, 90.5)
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Routing:
- net GND: track 332.1 -> 150.9 mm, vias 17 -> 4
- net +5V: track 246.5 -> 105.9 mm, vias 10 -> 1
- net /PB7: track 100.9 -> 0.00 mm, vias 4 -> 0
- net RESET1: track 137.8 -> 56.8 mm, vias 4 -> 2
- net RXD0: track 61.9 -> 0.00 mm, vias 2 -> 0
- net TXD0: track 61.8 -> 0.00 mm, vias 2 -> 0
- net Net-(U1-PE5): track 56.3 -> 0.00 mm, vias 2 -> 0
- net Net-(U1-PE4): track 52.9 -> 0.00 mm
- net /PH3: track 48.1 -> 0.00 mm, vias 2 -> 0
- net /PL1: track 46.6 -> 0.00 mm, vias 2 -> 0
- net Net-(U1-PE3): track 45.9 -> 0.00 mm, vias 2 -> 0
- net /PG5: track 45.6 -> 0.00 mm
- net /PH4: track 44.9 -> 0.00 mm, vias 2 -> 0
- net /PL0: track 38.9 -> 0.00 mm, vias 2 -> 0
- net VIN: track 99.0 -> 60.4 mm, vias 2 -> 1
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
Commit message: Update
Parts:
- moved PWM2 1.05 mm to (83.2, 105.8)
- moved PWM1 0.71 mm to (104.9, 105.8)
- moved ADC1 0.66 mm to (93.9, 154.2)
- moved ADC2 0.46 mm to (116.8, 154.2)
- moved COM1 0.24 mm to (126.6, 105.8)
- moved PWR1 0.16 mm to (76.5, 154.2)
Changed lines of the file:
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@@
 	(footprint "Connector_PinHeader_2.54mm:PinHeader_1x08_P2.54mm_Vertical"
 		(layer "F.Cu")
-		(at 116.825 153.7 90)
+		(at 116.825 154.16 90)
 		(descr "Through hole straight pin header, 1x08, 2.54mm pitch, single row")
 		(tags "Through hole pin header THT 1x08 2.54mm single row")
@@
 	(footprint "Connector_PinHeader_2.54mm:PinHeader_1x08_P2.54mm_Vertical"
 		(layer "F.Cu")
-		(at 93.94 153.5 90)
+		(at 93.94 154.16 90)
 		(descr "Through hole straight pin header, 1x08, 2.54mm pitch, single row")
 		(tags "Through hole pin header THT 1x08 2.54mm single row")
@@
 	(footprint "Connector_PinHeader_2.54mm:PinHeader_1x08_P2.54mm_Vertical"
 		(layer "F.Cu")
-		(at 104.16 105.7 -90)
+		(at 104.86 105.84 -90)
 		(descr "Through hole straight pin header, 1x08, 2.54mm pitch, single row")
 		(tags "Through hole pin header THT 1x08 2.54mm single row")
@@
 	(footprint "Connector_PinHeader_2.54mm:PinHeader_1x08_P2.54mm_Vertical"
 		(layer "F.Cu")
-		(at 126.36 105.7 -90)
+		(at 126.56 105.84 -90)
 		(descr "Through hole straight pin header, 1x08, 2.54mm pitch, single row")
 		(tags "Through hole pin header THT 1x08 2.54mm single row")
@@
 	(footprint "Connector_PinHeader_2.54mm:PinHeader_1x06_P2.54mm_Vertical"
 		(layer "F.Cu")
-		(at 76.45 154 90)
+		(at 76.45 154.16 90)
 		(descr "Through hole straight pin header, 1x06, 2.54mm pitch, single row")
 		(tags "Through hole pin header THT 1x06 2.54mm single row")
@@
 	(footprint "Connector_PinHeader_2.54mm:PinHeader_1x08_P2.54mm_Vertical"
 		(layer "F.Cu")
-		(at 82.18 105.6 -90)
+		(at 83.2 105.84 -90)
 		(descr "Through hole straight pin header, 1x08, 2.54mm pitch, single row")
 		(tags "Through hole pin header THT 1x08 2.54mm single row")
@@
 			"RCwCAABrnAAAAAAAALBjMUQsAgAAUwQAAAAAAAAQYzFELAIAAGucAAAAAAAA0GMxRCwCAABLBAAA"
 			"AAAAABBjMUQsAgAAa5wAAAAAAADwYzFELAIAABgAAAAAAAAAQCGE8f1/AAABAAAAAAAAAAAAAAAA"
-			"AAAA5iYAABsAAADmJgAAHgAAAAAAAAAAAAAAcGQxRCwCAAAAAAAAAA=="
+			"AAAA5iYAABsAAADmJgAAHgAAAAAAAAAAAAAAcGQxRCwCAAAAAAAAAAAAAAAAAAAAAAAAAAAAAAAA"
+			"AAAAAAAAAAAAAAAAAAAAAAAAAAAAAAAAAAAAAAAAAAAAAAAAAAAAAAAAAAAAAAAAAAAAAAAAAAAA"
+			"AAAAAAAAAAAAAAAAAAAAAAAAAAAAAAAAAAAAAAAAAAAAAAAAAAAAAAAAAAAAAAAAAAAAAAAAAAAA"
+			"AAAAAAAAAAAAAAAAAAAAAAAAAAAAAAAAAAAAAAAAAAAAAAAAAAAAAAAAAAAAAAAAAAAAAAAAAAAA"
+			"AAAAAAAAAAAAAAAAAAAAAAAAAAAAAAAAAAAAAAAAAAAAAAAAAAAAAAAAAAAAAAAAAAAAAAAAAAAA"
+			"AAAAAAAAAAAAAAAAAAAAAAAAAAAAAAAAAAAAAAAAAAAAAAAAAAAAAAAAAAAAAAAAAAAAAAAAAAAA"
+			"AAAAAAAAAAAAAAAAAAAAAAAAAAAAAAAAAAAAAAAAAAAAAAAAAAAAAAAAAAAAAAAAAAAAAAAAAAAA"
+			"AAAAAAAAAAAAAAAAAAAAAAAAAAAAAAAAAAAAAAAAAAAAAAAAAAAAAAAAAAAAAAAAAAAAAAAAAAAA"
+			"AAAAAAAAAAAAAAAAAAAAAAAAAAAAAAAAAAAAAAAAAAAAAAAAAAAAAAAAAAAAAAAAAAAAAAAAAAAA"
+			"AAAAAAAAAAAAAAAAAAAAAAAAAAAAAAAAAAAAAAAAAAAAAAAAAAAAAAAAAAAAAAAAAAAAAAAAAAAA"
+			"AAAAAAAAAAAAAAAAAAAAAAAAAAAAAAAAAAAAAAAAAAAAAAAAAAAAAAAAAAAAAAAAAAAAAAAAAAAA"
+			"AAAAAAAAAAAAAAAAAAAAAAAAAAAAAAAAAAAAAAAAAAAAAAAAAAAAAAAAAAAAAAAAAAAAAAAAAAAA"
+			"AAAAAAAAAAAAAAAAAAAAAAAAAAAAAAAAAAAAAAAAAAAAAAAAAAAAAAAAAAAAAAAAAAAAAAAAAAAA"
+			"AAAAAAAAAAAAAAAAAAAAAAAAAAAAAAAAAAAAAAAAAAAAAAAAAAAAAAAAAAAAAAAAAAAAAAAAAAAA"
+			"AAAAAAAAAAAAAAAAAAAAAAAAAAAAAAAAAAAAAAAAAAAAAAAAAAAAAAAAAAAAAAAAAAAAAAAAAAAA"
+			"AAAAAAAAAAAAAAAAAAAAAAAAAAAAAAAAAAAAAAAAAAAAAAAAAAAAAAAAAAAAAAAAAAAAAAAAAAAA"
+			"AAAAAAAAAAAAAAAAAAAAAAAAAAAAAAAAAAAAAAAAAAAAAAAAAAAAAAAAAAAAAAAAAAAAAAAAAAAA"
+			"AAAAAAAAAAAAAAAAAAAAAAAAAAAAAAAAAAAAAAAAAAAAAAAAAAAAAAAAAAAAAAAAAAAAAAAAAAAA"
+			"AAAAAAAAAAAAAAAAAAAAAAAAAAAAAAAAAAAAAAAAAAAAAAAAAAAAAA=="
 		)
 	)
 	(via
-		(at 137.72 154.13)
+		(at 137.82 154.16)
 		(size 3.5)
 		(drill 3)
@@
 	)
 	(via
-		(at 56.44 154.13)
+		(at 56.54 154.16)
 		(size 3.5)
 		(drill 3.2)
@@
 	)
 	(via
-		(at 131.37 105.87)
+		(at 131.47 105.84)
 		(size 3.5)
 		(drill 3)
@@
 	)
 	(via
-		(at 56.44 105.87)
+		(at 56.54 105.84)
 		(size 3.5)
 		(drill 3.2)

Commit message: Update
Parts:
- added J5: Conn_02x08, PCM_4ms_Connector:Pins_2x08_2.54mm_TH, F.Cu at (156.5, 133.3)
- moved J4 32.0 mm to (138.7, 148.9), turned to -90 degrees
- moved J3 26.4 mm to (136.1, 105.8), turned to 90 degrees
- moved ICSP2 13.0 mm to (87.3, 117.9)
- moved C16 5.88 mm to (165.7, 108.6), turned to 180 degrees
- moved RN11 4.26 mm to (73.4, 148.0)
- moved C1 4.16 mm to (73.4, 149.9)
- moved C17 3.97 mm to (162.2, 108.6)
- moved J1 3.62 mm to (137.4, 137.5)
- moved J2 3.19 mm to (137.4, 117.2)
- moved U2 2.87 mm to (84.3, 136.7)
- moved PWR1 2.15 mm to (74.3, 154.2)
- moved ADC2 1.83 mm to (115.0, 154.2)
- moved ADC1 1.78 mm to (92.2, 154.2)
- moved U1 1.20 mm to (106.3, 133.2), turned to 180 degrees
Connections:
- ADC1 pad 1: /ADC0 -> /ADC15
- ADC1 pad 2: /ADC1 -> /ADC14
- ADC1 pad 3: /ADC2 -> /ADC13
- ADC1 pad 4: /ADC3 -> /ADC12
- ADC1 pad 5: /ADC4 -> /ADC11
- ADC1 pad 6: /ADC5 -> /ADC10
- ADC1 pad 7: /ADC6 -> /ADC9
- ADC1 pad 8: /ADC7 -> /ADC8
- ADC2 pad 1: /ADC8 -> /ADC7
- ADC2 pad 2: /ADC9 -> /ADC6
- ADC2 pad 3: /ADC10 -> /ADC5
- ADC2 pad 4: /ADC11 -> /ADC4
- ADC2 pad 5: /ADC12 -> /ADC3
- ADC2 pad 6: /ADC13 -> /ADC2
- ADC2 pad 7: /ADC14 -> /ADC1
- ADC2 pad 8: /ADC15 -> /ADC0
- U1 pad 14: unconnected-(U1-PH2-Pad14) -> /PH2
- U1 pad 27: unconnected-(U1-PH7-Pad27) -> /PH7
- U1 pad 28: unconnected-(U1-PG3-Pad28) -> /PG3
- U1 pad 29: unconnected-(U1-PG4-Pad29) -> /PG4
- U1 pad 4: unconnected-(U1-PE2-Pad4) -> /PE2
- U1 pad 47: unconnected-(U1-PD4-Pad47) -> /PD4
- U1 pad 48: unconnected-(U1-PD5-Pad48) -> /PD5
- U1 pad 49: unconnected-(U1-PD6-Pad49) -> /PD6
- U1 pad 65: unconnected-(U1-PJ2-Pad65) -> /PJ2
- U1 pad 66: unconnected-(U1-PJ3-Pad66) -> /PJ3
- U1 pad 67: unconnected-(U1-PJ4-Pad67) -> /PJ4
- U1 pad 68: unconnected-(U1-PJ5-Pad68) -> /PJ5
- U1 pad 69: unconnected-(U1-PJ6-Pad69) -> /PJ6
- U1 pad 79: unconnected-(U1-PJ7-Pad79) -> /PJ7
- U1 pad 8: unconnected-(U1-PE6-Pad8) -> /PE6
- U1 pad 9: unconnected-(U1-PE7-Pad9) -> /PE7
Routing:
- net GND: track 150.9 -> 177.6 mm, vias 4 -> 5
- net VIN: track 60.4 -> 87.1 mm, vias 1 -> 2
- net +3V3: track 22.6 -> 43.7 mm, vias 1 -> 3
- net +5V: track 105.9 -> 126.6 mm
- net RESET1: track 56.8 -> 66.2 mm
- net Net-(D2-Pad2): track 34.9 -> 31.7 mm
