File: ArduinoMega2560/arduinomega_atmega8u2.kicad_sch (KiCad schematic)
At the start: 25 parts, among them J2 UJ2-BH-1-TH, U2 ATmega8U2-A, Y2 TSX-3225_16.0000MF18X-AC0

Commit message: Annotation problem
Parts:
- added C10: 100nF_0603_16V, PCM_4ms_Capacitor:C_0603, symbol PCM_4ms_Capacitor:100nF_0603_16V
- renumbered LED_RX1 to RX1, LED_TX1 to TX1
Connections:
- net at J2.4, JP_GND1.1 (A), L1.1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: now also C10.2
- net at U2.27 (UCAP): now also C10.1
Other:
- moved on the sheet: RN2A1, RN2D1
Changed lines of the file:
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@@
+    (stroke (width 0) (type default))
+  )
+  (wire (pts (xy 102.87 119.38) (xy 102.87 139.7))
     (stroke (width 0) (type default))
   )
@@
     (stroke (width 0) (type default))
   )
-  (wire (pts (xy 106.68 87.63) (xy 106.68 106.68))
+  (wire (pts (xy 99.06 87.63) (xy 99.06 106.68))
     (stroke (width 0) (type default))
   )
@@
     (stroke (width 0) (type default))
   )
-  (wire (pts (xy 60.96 95.25) (xy 90.17 95.25))
+  (wire (pts (xy 60.96 95.25) (xy 85.09 95.25))
     (stroke (width 0) (type default))
   )
@@
     (stroke (width 0) (type default))
   )
-  (wire (pts (xy 102.87 139.7) (xy 81.28 139.7))
-    (stroke (width 0) (type default))
-  )
   (wire (pts (xy 52.07 97.79) (xy 71.12 97.79))
     (stroke (width 0) (type default))
@@
     (stroke (width 0) (type default))
   )
+  (wire (pts (xy 111.76 92.71) (xy 102.87 92.71))
+    (stroke (width 0) (type default))
+  )
   (wire (pts (xy 60.96 128.27) (xy 71.12 128.27))
     (stroke (width 0) (type default))
@@
     (stroke (width 0) (type default))
   )
+  (wire (pts (xy 102.87 92.71) (xy 102.87 114.3))
+    (stroke (width 0) (type default))
+  )
   (wire (pts (xy 147.32 125.73) (xy 156.21 125.73))
     (stroke (width 0) (type default))
@@
     (stroke (width 0) (type default))
   )
-  (wire (pts (xy 101.6 85.09) (xy 101.6 95.25))
+  (wire (pts (xy 96.52 85.09) (xy 96.52 95.25))
     (stroke (width 0) (type default))
   )
@@
     (stroke (width 0) (type default))
   )
+  (wire (pts (xy 81.28 139.7) (xy 102.87 139.7))
+    (stroke (width 0) (type default))
+  )
   (wire (pts (xy 97.79 35.56) (xy 157.48 35.56))
     (stroke (width 0) (type default))
@@
     (stroke (width 0) (type default))
   )
-  (wire (pts (xy 111.76 85.09) (xy 101.6 85.09))
+  (wire (pts (xy 111.76 85.09) (xy 96.52 85.09))
     (stroke (width 0) (type default))
   )
@@
     (stroke (width 0) (type default))
   )
-  (wire (pts (xy 111.76 87.63) (xy 106.68 87.63))
-    (stroke (width 0) (type default))
-  )
-  (wire (pts (xy 101.6 95.25) (xy 97.79 95.25))
+  (wire (pts (xy 111.76 87.63) (xy 99.06 87.63))
+    (stroke (width 0) (type default))
+  )
+  (wire (pts (xy 96.52 95.25) (xy 92.71 95.25))
     (stroke (width 0) (type default))
   )
@@
     (stroke (width 0) (type default))
   )
-  (wire (pts (xy 97.79 106.68) (xy 106.68 106.68))
+  (wire (pts (xy 92.71 106.68) (xy 99.06 106.68))
     (stroke (width 0) (type default))
   )
@@
     (stroke (width 0) (type default))
   )
-  (wire (pts (xy 71.12 106.68) (xy 90.17 106.68))
+  (wire (pts (xy 71.12 106.68) (xy 85.09 106.68))
     (stroke (width 0) (type default))
   )
@@
   (symbol (lib_id "Device:LED") (at 189.23 120.65 0) (unit 1)
     (in_bom yes) (on_board yes) (dnp no)
-    (property "Reference" "LED_TX1" (at 187.6425 114.3 0)
+    (property "Reference" "TX1" (at 187.6425 114.3 0)
       (effects (font (size 1.27 1.27)))
     )
@@
       (project "ArduinoMega2560"
         (path "/9c604cc5-1a6f-41a9-b015-ecf51c009c14/42cc45d5-0d5b-4ebd-8f6c-e45958af00ea"
-          (reference "LED_TX1") (unit 1)
+          (reference "TX1") (unit 1)
         )
       )
@@
     )
   )
-  (symbol (lib_id "PCM_Resistor_AKL:R_0603") (at 93.98 106.68 90) (unit 1)
-    (in_bom yes) (on_board yes) (dnp no)
-    (property "Reference" "RN2A1" (at 93.98 100.33 90)
-      (effects (font (size 1.27 1.27)))
-    )
-    (property "Value" "22R_0603" (at 93.98 102.87 90)
-      (effects (font (size 1.27 1.27)) hide)
-    )
-    (property "Footprint" "PCM_Resistor_SMD_AKL:R_0603_1608Metric" (at 105.41 106.68 0)
-      (effects (font (size 1.27 1.27)) hide)
-    )
-    (property "Datasheet" "~" (at 93.98 106.68 0)
-      (effects (font (size 1.27 1.27)) hide)
-    )
-    (property "Display" "22R" (at 93.98 102.87 90)
+  (symbol (lib_id "PCM_Resistor_AKL:R_0603") (at 88.9 106.68 90) (unit 1)
+    (in_bom yes) (on_board yes) (dnp no)
+    (property "Reference" "RN2A1" (at 88.9 100.33 90)
+      (effects (font (size 1.27 1.27)))
+    )
+    (property "Value" "22R_0603" (at 88.9 102.87 90)
+      (effects (font (size 1.27 1.27)) hide)
+    )
+    (property "Footprint" "PCM_Resistor_SMD_AKL:R_0603_1608Metric" (at 100.33 106.68 0)
+      (effects (font (size 1.27 1.27)) hide)
+    )
+    (property "Datasheet" "~" (at 88.9 106.68 0)
+      (effects (font (size 1.27 1.27)) hide)
+    )
+    (property "Display" "22R" (at 88.9 102.87 90)
       (effects (font (size 1.27 1.27)))
     )
@@
   (symbol (lib_id "Device:LED") (at 189.23 107.95 0) (unit 1)
     (in_bom yes) (on_board yes) (dnp no) (fields_autoplaced)
-    (property "Reference" "LED_RX1" (at 187.6425 101.6 0)
+    (property "Reference" "RX1" (at 187.6425 101.6 0)
       (effects (font (size 1.27 1.27)))
     )
@@
       (project "ArduinoMega2560"
         (path "/9c604cc5-1a6f-41a9-b015-ecf51c009c14/42cc45d5-0d5b-4ebd-8f6c-e45958af00ea"
-          (reference "LED_RX1") (unit 1)
+          (reference "RX1") (unit 1)
         )
       )
@@
     )
   )
-  (symbol (lib_id "PCM_Resistor_AKL:R_0603") (at 93.98 95.25 270) (unit 1)
-    (in_bom yes) (on_board yes) (dnp no)
-    (property "Reference" "RN2D1" (at 93.98 88.9 90)
-      (effects (font (size 1.27 1.27)))
-    )
-    (property "Value" "22R_0603" (at 93.98 91.44 90)
-      (effects (font (size 1.27 1.27)) hide)
-    )
-    (property "Footprint" "PCM_Resistor_SMD_AKL:R_0603_1608Metric" (at 82.55 95.25 0)
-      (effects (font (size 1.27 1.27)) hide)
-    )
-    (property "Datasheet" "~" (at 93.98 95.25 0)
-      (effects (font (size 1.27 1.27)) hide)
-    )
-    (property "Display" "22R" (at 93.98 91.44 90)
+  (symbol (lib_id "PCM_Resistor_AKL:R_0603") (at 88.9 95.25 270) (unit 1)
+    (in_bom yes) (on_board yes) (dnp no)
+    (property "Reference" "RN2D1" (at 88.9 88.9 90)
+      (effects (font (size 1.27 1.27)))
+    )
+    (property "Value" "22R_0603" (at 88.9 91.44 90)
+      (effects (font (size 1.27 1.27)) hide)
+    )
+    (property "Footprint" "PCM_Resistor_SMD_AKL:R_0603_1608Metric" (at 77.47 95.25 0)
+      (effects (font (size 1.27 1.27)) hide)
+    )
+    (property "Datasheet" "~" (at 88.9 95.25 0)
+      (effects (font (size 1.27 1.27)) hide)
+    )
+    (property "Display" "22R" (at 88.9 91.44 90)
       (effects (font (size 1.27 1.27)))
     )
@@
         )
       )
+    )
+  )
+  (symbol (lib_id "PCM_4ms_Capacitor:100nF_0603_16V") (at 102.87 116.84 0) (unit 1)
+    (in_bom yes) (on_board yes) (dnp no)
+    (property "Reference" "C10" (at 105.41 115.5763 0)
+      (effects (font (size 1.27 1.27)) (justify left))
+    )
+    (property "Value" "100nF_0603_16V" (at 102.87 113.03 0)
+      (effects (font (size 1.27 1.27)) hide)
+    )
+    (property "Footprint" "PCM_4ms_Capacitor:C_0603" (at 100.33 121.92 0)
+      (effects (font (size 1.27 1.27)) (justify left) hide)
+    )
+    (property "Datasheet" "" (at 102.87 116.84 0)
+      (effects (font (size 1.27 1.27)) hide)
+    )
+    (property "Specifications" "0.1uF, Min. 16V 10%, X7R or X5R or similar" (at 100.33 124.714 0)
+      (effects (font (size 1.27 1.27)) (justify left) hide)
+    )
+    (property "Manufacturer" "AVX Corporation" (at 100.33 126.238 0)
+      (effects (font (size 1.27 1.27)) (justify left) hide)
+    )
+    (property "Part Number" "0603YC104KAT2A" (at 100.33 127.762 0)
+      (effects (font (size 1.27 1.27)) (justify left) hide)
+    )
+    (property "Display" "1uF" (at 105.41 118.1163 0)
+      (effects (font (size 1.27 1.27)) (justify left))
+    )
+    (property "JLCPCB ID" "C14663" (at 104.14 129.54 0)
+      (effects (font (size 1.27 1.27)) hide)
+    )
+    (pin "2")
+    (pin "1")
+    (instances
+      (project "ArduinoMega2560"
+        (path "/9c604cc5-1a6f-41a9-b015-ecf51c009c14/42cc45d5-0d5b-4ebd-8f6c-e45958af00ea"
+          (reference "C10") (unit 1)
+        )
+      )

Commit message: Update label
Parts:
- renumbered RN2A1 to RN21, RN2D1 to RN24, RN4A1 to RN41, RN4B1 to RN42, RN4C1 to RN43, RN4D1 to RN44, RN5A1 to RN51
Connections:
- net RESET renamed RESET1
Changed lines of the file:
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@@
 		)
 	)
-	(hierarchical_label "RESET"
+	(global_label "USBVCC"
 		(shape input)
-		(at 190.5 143.51 0)
+		(at 120.65 57.15 180)
+		(fields_autoplaced yes)
 		(effects
 			(font
 				(size 1.27 1.27)
 			)
-			(justify left)
-		)
-	)
-	(hierarchical_label "USBVCC"
+			(justify right)
+		)
+		(property "Intersheetrefs" "${INTERSHEET_REFS}"
+			(at 110.2262 57.15 0)
+			(effects
+				(font
+					(size 1.27 1.27)
+				)
+				(justify right)
+				(hide yes)
+			)
+		)
+	)
+	(global_label "USBVCC"
 		(shape input)
-		(at 120.65 57.15 180)
+		(at 34.29 63.5 0)
+		(fields_autoplaced yes)
 		(effects
 			(font
 				(size 1.27 1.27)
 			)
-			(justify right)
-		)
-	)
-	(hierarchical_label "USBVCC"
+			(justify left)
+		)
+		(property "Intersheetrefs" "${INTERSHEET_REFS}"
+			(at 44.7138 63.5 0)
+			(effects
+				(font
+					(size 1.27 1.27)
+				)
+				(justify left)
+				(hide yes)
+			)
+		)
+	)
+	(global_label "RESET2"
 		(shape input)
-		(at 34.29 63.5 0)
+		(at 72.39 50.8 180)
+		(fields_autoplaced yes)
 		(effects
 			(font
 				(size 1.27 1.27)
 			)
+			(justify right)
+		)
+		(property "Intersheetrefs" "${INTERSHEET_REFS}"
+			(at 62.4502 50.8 0)
+			(effects
+				(font
+					(size 1.27 1.27)
+				)
+				(justify right)
+				(hide yes)
+			)
+		)
+	)
+	(global_label "RESET1"
+		(shape input)
+		(at 190.5 143.51 0)
+		(fields_autoplaced yes)
+		(effects
+			(font
+				(size 1.27 1.27)
+			)
 			(justify left)
+		)
+		(property "Intersheetrefs" "${INTERSHEET_REFS}"
+			(at 200.4398 143.51 0)
+			(effects
+				(font
+					(size 1.27 1.27)
+				)
+				(justify left)
+				(hide yes)
+			)
 		)
 	)
@@
 		)
 	)
-	(hierarchical_label "RESET2"
-		(shape input)
-		(at 72.39 50.8 180)
-		(effects
-			(font
-				(size 1.27 1.27)
-			)
-			(justify right)
-		)
-	)
 	(hierarchical_label "PE1"
 		(shape input)
@@
 		(on_board yes)
 		(dnp no)
-		(property "Reference" "RN4C1"
+		(property "Reference" "RN43"
 			(at 199.39 115.57 90)
 			(effects
@@
 			(project "ArduinoMega2560"
 				(path "/9c604cc5-1a6f-41a9-b015-ecf51c009c14/42cc45d5-0d5b-4ebd-8f6c-e45958af00ea"
-					(reference "RN4C1")
+					(reference "RN43")
 					(unit 1)
 				)
@@
 		(on_board yes)
 		(dnp no)
-		(property "Reference" "RN4B1"
+		(property "Reference" "RN42"
 			(at 187.96 90.17 90)
 			(effects
@@
 			(project "ArduinoMega2560"
 				(path "/9c604cc5-1a6f-41a9-b015-ecf51c009c14/42cc45d5-0d5b-4ebd-8f6c-e45958af00ea"
-					(reference "RN4B1")
+					(reference "RN42")
 					(unit 1)
 				)
@@
 		(on_board yes)
 		(dnp no)
-		(property "Reference" "RN2A1"
+		(property "Reference" "RN21"
 			(at 88.9 100.33 90)
 			(effects
@@
 			(project "ArduinoMega2560"
 				(path "/9c604cc5-1a6f-41a9-b015-ecf51c009c14/42cc45d5-0d5b-4ebd-8f6c-e45958af00ea"
-					(reference "RN2A1")
+					(reference "RN21")
 					(unit 1)
 				)
@@
 		(on_board yes)
 		(dnp no)
-		(property "Reference" "RN4D1"
+		(property "Reference" "RN44"
 			(at 199.39 102.87 90)
 			(effects
@@
 			(project "ArduinoMega2560"
 				(path "/9c604cc5-1a6f-41a9-b015-ecf51c009c14/42cc45d5-0d5b-4ebd-8f6c-e45958af00ea"
-					(reference "RN4D1")
+					(reference "RN44")
 					(unit 1)
 				)
@@
 		(on_board yes)
 		(dnp no)
-		(property "Reference" "RN4A1"
+		(property "Reference" "RN41"
 			(at 187.96 81.28 90)
 			(effects
@@
 			(project "ArduinoMega2560"
 				(path "/9c604cc5-1a6f-41a9-b015-ecf51c009c14/42cc45d5-0d5b-4ebd-8f6c-e45958af00ea"
-					(reference "RN4A1")
+					(reference "RN41")
 					(unit 1)
 				)
@@
 		(on_board yes)
 		(dnp no)
-		(property "Reference" "RN2D1"
+		(property "Reference" "RN24"
 			(at 88.9 88.9 90)
 			(effects
@@
 			(project "ArduinoMega2560"
 				(path "/9c604cc5-1a6f-41a9-b015-ecf51c009c14/42cc45d5-0d5b-4ebd-8f6c-e45958af00ea"
-					(reference "RN2D1")
+					(reference "RN24")
 					(unit 1)
 				)
@@
 		(on_board yes)
 		(dnp no)
-		(property "Reference" "RN5A1"
+		(property "Reference" "RN51"
 			(at 110.49 43.18 0)
 			(effects
@@
 			(project "ArduinoMega2560"
 				(path "/9c604cc5-1a6f-41a9-b015-ecf51c009c14/42cc45d5-0d5b-4ebd-8f6c-e45958af00ea"
-					(reference "RN5A1")
-					(unit 1)
-				)
+					(reference "RN51")
+					(unit 1)
+				)

Commit message: Update Trace
Parts:
- renumbered J2 to USB1
Changed lines of the file:
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@@
 		(dnp no)
 		(fields_autoplaced yes)
-		(property "Reference" "J2"
+		(property "Reference" "USB1"
 			(at 43.18 87.63 0)
 			(effects
@@
 			(project "ArduinoMega2560"
 				(path "/9c604cc5-1a6f-41a9-b015-ecf51c009c14/42cc45d5-0d5b-4ebd-8f6c-e45958af00ea"
-					(reference "J2")
+					(reference "USB1")
 					(unit 1)
 				)

Commit message: Update tracing
Connections:
- net RESET1: now also RESET_EN1.1 (A); no longer RESET_EN1.2 (B)
- net at C7.2: now also RESET_EN1.2 (B); no longer RESET_EN1.1 (A)
Changed lines of the file:
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@@
 	(wire
 		(pts
-			(xy 69.85 78.74) (xy 69.85 80.01)
+			(xy 165.1 143.51) (xy 173.99 143.51)
 		)
 		(stroke
@@
 	(wire
 		(pts
-			(xy 71.12 124.46) (xy 71.12 128.27)
+			(xy 69.85 78.74) (xy 69.85 80.01)
 		)
 		(stroke
@@
 	(wire
 		(pts
-			(xy 147.32 120.65) (xy 185.42 120.65)
+			(xy 71.12 124.46) (xy 71.12 128.27)
 		)
 		(stroke
@@
 	(wire
 		(pts
-			(xy 181.61 143.51) (xy 190.5 143.51)
+			(xy 147.32 120.65) (xy 185.42 120.65)
 		)
 		(stroke
@@
 	(wire
 		(pts
+			(xy 181.61 143.51) (xy 190.5 143.51)
+		)
+		(stroke
+			(width 0)
+			(type default)
+		)
+	)
+	(wire
+		(pts
 			(xy 77.47 33.02) (xy 81.28 33.02)
 		)
@@
 	(wire
 		(pts
-			(xy 165.1 143.51) (xy 173.99 143.51)
-		)
-		(stroke
-			(width 0)
-			(type default)
-		)
-	)
-	(wire
-		(pts
 			(xy 156.21 125.73) (xy 156.21 143.51)
 		)
@@
 		(lib_id "Jumper:SolderJumper_2_Open")
 		(at 177.8 143.51 0)
-		(mirror x)
+		(mirror y)
 		(unit 1)
 		(exclude_from_sim no)
@@
 		(dnp no)
 		(property "Reference" "RESET_EN1"
-			(at 177.8 149.86 0)
+			(at 177.546 147.066 0)
 			(effects
 				(font
@@
 		)
 		(property "Value" "SolderJumper_2_Open"
-			(at 177.8 147.32 0)
+			(at 177.546 149.606 0)
 			(effects
 				(font

Commit message: Update trace
Parts:
- added C16, C17: 22pF_0603_16V, PCM_4ms_Capacitor:C_0603, symbol PCM_4ms_Capacitor:100nF_0603_16V
- added Q1: Crystal_16MHz, Crystal:Crystal_HC49-4H_Vertical, symbol PCM_SL_Devices:Crystal_16MHz
Connections:
- net GND: now also C16.2, C17.2
- net XT1: now reaches R2.2, R4.1, Y2.1
- net XT1: now also C16.1, Q1.2
- net XT2: now reaches R2.1, U2.2 (PC0/XTAL2), Y2.3
- net XT2: now also C17.1, Q1.1

Commit message: Update
Using Rev3
Parts:
- removed C16, C17: 22pF_0603_16V, PCM_4ms_Capacitor:C_0603, symbol PCM_4ms_Capacitor:100nF_0603_16V
- removed D2, D3: PGB1010603MR, Littelfuse_DiodeZ-TVS-PGB1010603MR:DIOC1608X36N, symbol Littelfuse_DiodeZ-TVS-PGB1010603MR:PGB1010603MR
- removed F1: C2Q 500mA, BelFuse_C2Q500:C2_BEL, symbol BelFuse_C2Q500:C2Q_500
- removed L1: BLM21PG221SN1D, Murata_BLM21PG221SN1D:IND_BLM21_MUR, symbol Murata_BLM21PG221SN1D:BLM21PG221SN1D
- removed Q1: Crystal_16MHz, Crystal:Crystal_HC49-4H_Vertical, symbol PCM_SL_Devices:Crystal_16MHz
- removed R4: 27R_0603, PCM_Resistor_SMD_AKL:R_0603_1608Metric, symbol PCM_Resistor_AKL:R_0603
- removed Y2: TSX-3225_16.0000MF18X-AC0, EPSON_TSX-3225-16MF18X-AC0:XTAL_TSX-3225_16.0000MF18X-AC0, symbol EPSON-TSX-3225-16MF18X-AC0:TSX-3225_16.0000MF18X-AC0
- added C14, C15: 100nF_0603_16V, PCM_4ms_Capacitor:C_0603, symbol PCM_4ms_Capacitor:100nF_0603_16V
- added D2: CD1206-S01575, Diode_CD1206-S01575_Bourns:DIODE_CD1206-S01575_BRN, symbol Diode_CD1206-S01575_Bourns:CD1206-S01575
- added F1: MF-MSMF050-2, Fuse_MF-MSMF050-2_Bourns:FUSE_F050-2, symbol Fuse_MF-MSMF050-2_Bourns:MF-MSMF050-2
- added J6: PINHD_2x2_Male, Connector_PinHeader_2.54mm:PinHeader_2x02_P2.54mm_Vertical, symbol PCM_SL_Pin_Headers:PINHD_2x2_Male
- added L1: MH2029-300Y, FerriteBead_MH2029-300Y_Bourns:IND_BOURNS_MH2029, symbol FerriteBead_MH2029-300Y_Bourns:MH2029-300Y
- added RN34: 1K_0603, PCM_Resistor_SMD_AKL:R_0603_1608Metric, symbol PCM_Resistor_AKL:R_0603
- added Y2: Crystal_16MHz, Crystal:Crystal_HC49-4H_Vertical, symbol PCM_SL_Devices:Crystal_16MHz
- added Z1, Z2: CG0603MLC-05E, Varistor_CG0603MLC-05E_Bourns:VARC1608X56N, symbol Varistor_CG0603MLC-05E_Bourns:CG0603MLC-05E
- renumbered ICSP1 to ICSP2, RN51 to RN52
Connections:
- net +5V: now also D2.1
- net GND: now also C14.1, C15.1, RN34.2
- net RESET2: now also D2.2
- net USBVCC: now also F1.2
- net XT1: now also U2.1 (XTAL1), C15.2, Y2.1
- net XT2: now also C14.2, Y2.2
- net at C10.2, JP_GND1.1 (A), U2.28 (UGND)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: now also L1.2
- net at C7.1, U2.13 (~{HWB}/PD7), UBOOT1.2 (B): now also RN34.1
- net at C8.1, USB1.1: now also F1.1
- net at RN21.1, USB1.2: now also Z1.1
- net at RN24.2, USB1.3: now also Z2.1
- net at USB1.5 (SHIELD), USB1.6 (SHIELD): now also L1.1, Z1.2, Z2.2
- net PB4: now reaches U2.18 (PB4)
- net PB4: now also J6.1
- net PB5: now reaches U2.19 (PB5)
- net PB5: now also J6.3
- net PB6: now reaches U2.20 (PB6)
- net PB6: now also J6.2
- net PB7: now reaches U2.21 (PB7)
- net PB7: now also J6.4
- net MISO renamed MISO2
- net MOSI renamed MOSI2
- net SCK renamed SCK2
Other:
- moved on the sheet: C8, ICSP2, R2, RN21, RN24, RN52, USB1
