File: ArduinoMega2560/Excluded.kicad_sch (KiCad schematic)
At the start: 0 parts

Commit message: Update footprint and silkscree
next, fixing the trace on the pinheader
Parts:
- added J3, J4: PINHD_1x2_Female, Connector_PinSocket_2.54mm:PinSocket_1x02_P2.54mm_Vertical, symbol PCM_SL_Pin_Headers:PINHD_1x2_Female
- added J5: Conn_02x08, PCM_4ms_Connector:Pins_2x08_2.54mm_TH, symbol PCM_4ms_Connector:Conn_02x08
Connections:
- new net +5V: J3.1, J3.2
- new net GND: J4.1, J4.2
- new net PD4: J5.2 (P2)
- new net PD5: J5.4 (P4)
- new net PD6: J5.6 (P6)
- new net PE2: J5.8 (+12V)
- new net PE6: J5.10 (GND)
- new net PE7: J5.12 (GND)
- new net PG3: J5.14 (-12V)
- new net PG4: J5.16 (P16)
- new net PH2: J5.13 (-12)
- new net PH7: J5.15 (-12V)

Commit message: Update Eth
Parts:
- removed J3, J4: PINHD_1x2_Female, Connector_PinSocket_2.54mm:PinSocket_1x02_P2.54mm_Vertical, symbol PCM_SL_Pin_Headers:PINHD_1x2_Female
