File: ArduinoMega2560/arduinomega_power.kicad_sch (KiCad schematic)
At the start: 17 parts, among them T1 PMV48XP_215, U3 LMV358IDGK

Commit message: Update shield
Parts:
- Cp1, Cp2: Display 47uF -> 47uF 16V
Changed lines of the file:
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@@
 			)
 		)
-		(property "Display" "47uF"
+		(property "Display" "47uF 16V"
 			(at 59.69 66.04 90)
 			(effects
@@
 			)
 		)
-		(property "Display" "47uF"
+		(property "Display" "47uF 16V"
 			(at 127 66.04 90)
 			(effects
