File: Arduino_Shield_PoEth-Wifi-GSM/PowerOverEthernet.kicad_sch (KiCad schematic)
At the start: 61 parts, among them Q2 Crsytal 25MHz 6pF 150Ohm 4-pi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, U1 CAT811TTBI-GT3, U1 W5500, U3 SN74LVC1G125DBVR, U4 LP2986AILD-3.3/NOPB

Commit message: Checking Eth PoE
Parts:
- removed Q2: Crsytal 25MHz 6pF 150Ohm 4-pin SMD, Murata_XRCGB25M000F3M00R0:XRCGB27M120F3M10R0_MUR, symbol Murata_XRCGB25M000F3M00R0:Crsytal 25MHz 6pF 150Ohm 4-pin SMD
- removed R13, R21: 0R_0603, PCM_Resistor_SMD_AKL:R_0603_1608Metric, symbol PCM_Resistor_AKL:R_0603
- added RN32, RN33, RN34: 10K_0603, PCM_Resistor_SMD_AKL:R_0603_1608Metric, symbol PCM_Resistor_AKL:R_0603
- added X2: 25MHz 18pF, Crystal_25MHz_AbraconLLC:XTAL_HC49P488W46L1150T500H350, symbol Crystal_25MHz_AbraconLLC:ABL-25.000MHZ-B2F
- C36: Display 0.1uF -> 10nF
- renumbered C36 to C19, C32 to C31, C31 to C32, ICSP to ICSP1, RN1A to RN11, RN1B to RN12, RN1C to RN13, RN1D to RN14, RN2A to RN21, RN2B to RN22, RN2C to RN23, RN2D to RN24, RN3D to RN31, RN3B to RN3B1, RN3C to RN3C1, RN4A to RN41, RN4B to RN42, RN4D to RN44, SW_RESET to SW_RESET1
Connections:
- net +3V3D: now also RN32.1, RN33.1, RN34.1
- net GND_3V3: now also C35.1; no longer C35.2
- net PMODE0: no longer U1.45 (PMODE0)
- net PMODE1: no longer U1.44 (PMODE1)
- net PMODE2: no longer U1.43 (PMODE2)
- net RXN1: now reaches RN13.1, U1.5 (RXN)
- net TXN1: now reaches RN11.1, U1.1 (TXN)
- net TXP1: now reaches RN12.1, U1.2 (TXP)
- net at U1.20 (TOCAP): now also C35.2
- net at C36.1, U1.22 (1V2O): no longer C35.1
- net RSVD6: now reaches RN42.1, U1.23 (RSVD)
- net RXP1: now reaches RN14.1, U1.6 (RXP)
- net XI: no longer names the net of C34.1, R45.2, U1.30 (XI/CLKIN)
- net XI: now also X2.1
- net XO: no longer names the net of C33.1, R45.1, U1.31 (XO)
- net XO: now also X2.2
- new net: RN33.2, U1.44 (PMODE1)
- new net: RN32.2, U1.45 (PMODE0)
- new net: RN34.2, U1.43 (PMODE2)
Other:
- moved on the sheet: C20, C21, C24, C25, C28, C29, C30, C31, C32, C33, C34, C35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

Commit message: Tuning serial and crystal tracks
Parts:
- removed C37, C38: 22uF_16V, Capacitor_THT:CP_Radial_D4.0mm_P1.50mm, symbol PCM_SL_Capacitors:22uF_16V
- removed ICSP1: PINHD_2x3_Male, Connector_PinHeader_2.54mm:PinHeader_2x03_P2.54mm_Vertical, symbol PCM_SL_Pin_Headers:PINHD_2x3_Male
- removed L1, L2: FerriteBead_0603_1.5A, PCM_4ms_Resistor:R_0603, symbol PCM_4ms_Inductor:FerriteBead_0603_1.5A
- removed R11, R15, R20: R_DNP, PCM_4ms_Resistor:R_0603, symbol PCM_4ms_Resistor:R_DNP
- removed R9, RN3B1, RN3C1: 10K_0603, PCM_Resistor_SMD_AKL:R_0603_1608Metric, symbol PCM_Resistor_AKL:R_0603
- removed SW_RESET1: Push_Button, Button_Switch_THT:SW_PUSH_6mm, symbol PCM_SL_Devices:Push_Button
- removed U1: CAT811TTBI-GT3, Package_TO_SOT_SMD:SOT-143, symbol Power_Supervisor:CAT811TTBI-GT3
- removed U3: SN74LVC1G125DBVR, TI_SN74LVC1G125DBVR:DBV0005A_L, symbol TI_SN74LVC1G125DBVR:SN74LVC1G125DBVR
- added J?: PINHD_2x4_Male, Connector_PinHeader_2.54mm:PinHeader_2x04_P2.54mm_Vertical, symbol PCM_SL_Pin_Headers:PINHD_2x4_Male
- added L?: MH2029-300Y, FerriteBead_MH2029-300Y_Bourns:IND_BOURNS_MH2029, symbol FerriteBead_MH2029-300Y_Bourns:MH2029-300Y
Connections:
- net GND_12V is gone; now on net GND: RJ45.10 (V-)
- net GND_3V3 is gone; now on net GND: C1.1, C10.1, C16.1, C19.1, C20.2, C21.2, C24.2, C25.2, C28.2, C29.2, C30.2, C31.2, C32.2, C33.2, C34.2, C35.1, C36.2, R46.2, RN21.2, RN22.2, RN23.2, RN24.2, RN41.2, RN42.2, U1.14 (AGND), U1.16 (AGND), U1.19 (AGND), U1.3 (AGND), U1.48 (AGND), U1.9 (AGND)
- net GND: now also U1.29 (GND)
- net Earth renamed EARTH
Other:
- moved on the sheet: C1, C10, C16, C17, C18, C19, C20, C21, C24, C25, C28, C29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

Commit message: Update Eth
Parts:
- removed J?: PINHD_2x4_Male, Connector_PinHeader_2.54mm:PinHeader_2x04_P2.54mm_Vertical, symbol PCM_SL_Pin_Headers:PINHD_2x4_Male
- removed L?: MH2029-300Y, FerriteBead_MH2029-300Y_Bourns:IND_BOURNS_MH2029, symbol FerriteBead_MH2029-300Y_Bourns:MH2029-300Y
Changed lines of the file:
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@@
 		(on_board yes)
 		(dnp no)
-		(fields_autoplaced yes)
 		(property "Reference" "#PWR025"
 			(at 337.82 199.39 0)
@@
 		)
 		(property "Value" "EARTH"
-			(at 340.36 194.3099 0)
+			(at 334.772 197.612 0)
 			(effects
 				(font
@@
 					(unit 1)
 				)
-			)
-		)
-	)
-	(symbol
-		(lib_id "FerriteBead_MH2029-300Y_Bourns:MH2029-300Y")
-		(at 340.36 207.01 0)
-		(unit 1)
-		(exclude_from_sim no)
-		(in_bom yes)
-		(on_board yes)
-		(dnp no)
-		(fields_autoplaced yes)
-		(property "Reference" "L?"
-			(at 347.98 199.39 0)
-			(effects
-				(font
-					(size 1.524 1.524)
-				)
-			)
-		)
-		(property "Value" "MH2029-300Y"
-			(at 347.98 201.93 0)
-			(effects
-				(font
-					(size 1.524 1.524)
-				)
-			)
-		)
-		(property "Footprint" "FerriteBead_MH2029-300Y_Bourns:IND_BOURNS_MH2029"
-			(at 348.234 212.09 0)
-			(effects
-				(font
-					(size 1.27 1.27)
-					(italic yes)
-				)
-				(hide yes)
-			)
-		)
-		(property "Datasheet" "MH2029-300Y"
-			(at 348.234 214.122 0)
-			(effects
-				(font
-					(size 1.27 1.27)
-					(italic yes)
-				)
-				(hide yes)
-			)
-		)
-		(property "Description" "30 Ohms @ 100 MHz 1 Power, Signal Line Ferrite Bead 0805 (2012 Metric) 3A 25mOhm"
-			(at 348.488 216.408 0)
-			(effects
-				(font
-					(size 1.27 1.27)
-				)
-				(hide yes)
-			)
-		)
-		(pin "2"
-		)
-		(pin "1"
-		)
-		(instances
-			(project ""
-				(path "/00744368-faf2-4f6e-8fde-6584e08422b6/8c23214b-35e1-4477-9fe9-7ddb9ea6380c"
-					(reference "L?")
-					(unit 1)
-				)
-			)
-		)
-	)
-	(symbol
-		(lib_id "PCM_SL_Pin_Headers:PINHD_2x4_Male")
-		(at 85.09 138.43 0)
-		(unit 1)
-		(exclude_from_sim no)
-		(in_bom yes)
-		(on_board yes)
-		(dnp no)
-		(fields_autoplaced yes)
-		(property "Reference" "J?"
-			(at 85.09 128.27 0)
-			(effects
-				(font
-					(size 1.27 1.27)
-				)
-			)
-		)
-		(property "Value" "PINHD_2x4_Male"
-			(at 85.09 130.81 0)
-			(effects
-				(font
-					(size 1.27 1.27)
-				)
-			)
-		)
-		(property "Footprint" "Connector_PinHeader_2.54mm:PinHeader_2x04_P2.54mm_Vertical"
-			(at 85.09 127 0)
-			(effects
-				(font
-					(size 1.27 1.27)
-				)
-				(hide yes)
-			)
-		)
-		(property "Datasheet" ""
-			(at 83.82 128.27 0)
-			(effects
-				(font
-					(size 1.27 1.27)
-				)
-				(hide yes)
-			)
-		)
-		(property "Description" "Pin Header male with pin space 2.54mm. Pin Count -8"
-			(at 85.09 138.43 0)
-			(effects
-				(font
-					(size 1.27 1.27)
-				)
-				(hide yes)
-			)
-		)
-		(pin "3"
-		)
-		(pin "2"
-		)
-		(pin "4"
-		)
-		(pin "6"
-		)
-		(pin "8"
-		)
-		(pin "7"
-		)
-		(pin "5"
-		)
-		(pin "1"
-		)
-		(instances
-			(project ""
-				(path "/00744368-faf2-4f6e-8fde-6584e08422b6/8c23214b-35e1-4477-9fe9-7ddb9ea6380c"
-					(reference "J?")
-					(unit 1)
-				)
