File: Arduino_Shield_PoE-Wifi/Wifi.kicad_sch (KiCad schematic)
At the start: 12 parts, among them U2 74HC245

Commit message: Update
Parts:
- added JP1, JP2, JP3, JP4, JP5, JP6: SolderJumper_2_Open, Connector_PinHeader_2.54mm:PinHeader_1x02_P2.54mm_Vertical, symbol Jumper:SolderJumper_2_Open
- gave numbers to parts that had none: 1
- renumbered LED_ACT to LED_ACT1, LED_ERR to LED_ERR1, LED_WIFI to LED_WIFI1, U2 to U3
Connections:
- net RXD_5V is gone; now on net WAKE_5V: U3.9 (A7)
- net CS_3V3: now also JP2.2 (B)
- net GND: no longer U2.12 (GND_2), U2.28 (GND_3), U2.9 (GND_1), U3.10 (GND), U3.19 (CE)
- net IRQ: now also JP5.1 (A); no longer U2.13 (IRQN)
- net MOSI_3V3: now also JP1.2 (B)
- net RST_3V3: now also JP6.1 (A); no longer U2.4 (RESET_N)
- net SCK_3V3: now also JP4.2 (B); no longer U2.18 (SPI_SCK)
- net WAKE_3V3: now also U3.11 (B7); no longer U3.17 (B1)
- net WAKE_5V: no longer U3.3 (A1)
- net at U2.16 (SPI_SSN): now also JP2.1 (A)
- net +3V3_2 renamed +3V3C
- net RXD_3V3: no longer names the net of U2.15 (SPI_RXD)
- net RXD_3V3: now also JP1.1 (A); no longer U3.11 (B7)
- net TXD: no longer names the net of U2.17 (SPI_TXD)
- net TXD: now also JP3.1 (A)
- new net: JP6.2 (B), U2.4 (RESET_N)
- new net: JP5.2 (B), U2.13 (IRQN)
- new net: JP4.1 (A), U2.18 (SPI_SCK)
- new net GNDC: U2.12 (GND_2), U2.28 (GND_3), U2.9 (GND_1), U3.10 (GND), U3.19 (CE)
- new net MISO_3V3: JP3.2 (B), U3.17 (B1)
- new net MISO_5V: U3.3 (A1)
Other:
- moved on the sheet: LED_ACT1, LED_ERR1, LED_WIFI1, RG81, RG82, RG83, RG84, RG85, RG86, RG87, U2

Commit message: fixing schematics
Fix using ESP8266 12-E
Parts:
- renumbered U2 to U3, U3 to U4
Changed lines of the file:
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@@
 		(dnp no)
 		(fields_autoplaced yes)
-		(property "Reference" "U2"
+		(property "Reference" "U3"
 			(at 88.9 113.03 0)
 			(effects
@@
 			(project ""
 				(path "/00744368-faf2-4f6e-8fde-6584e08422b6/5238eee7-729f-4732-95e2-6eb150e234ab"
-					(reference "U2")
+					(reference "U3")
 					(unit 1)
 				)
@@
 		(dnp no)
 		(fields_autoplaced yes)
-		(property "Reference" "U3"
+		(property "Reference" "U4"
 			(at 103.7433 43.18 0)
 			(effects
@@
 			(project ""
 				(path "/00744368-faf2-4f6e-8fde-6584e08422b6/5238eee7-729f-4732-95e2-6eb150e234ab"
-					(reference "U3")
-					(unit 1)
-				)
+					(reference "U4")
+					(unit 1)
+				)
