File: Arduino_Shield_PoE-Wifi/arduinomega_power.kicad_sch (KiCad schematic)
At the start: 20 parts, among them T1 PMV48XP_215, U3 LMV358IDGK

Commit message: Update
Parts:
- removed C12, C13: 100nF_0603_16V, PCM_4ms_Capacitor:C_0603, symbol PCM_4ms_Capacitor:100nF_0603_16V
- removed Cp1, Cp2: 47uF_10V, Capacitor_THT:CP_Radial_D4.0mm_P1.50mm, symbol PCM_SL_Capacitors:47uF_10V
- removed LED_PB7: LED_0805_Yellow, PCM_LED_SMD_AKL:LED_0805_2012Metric, symbol PCM_LED_AKL:LED_0805_Yellow
- removed RN36: 1K_0603, PCM_Resistor_SMD_AKL:R_0603_1608Metric, symbol PCM_Resistor_AKL:R_0603
- removed RN53, RN54: 10K_0603, PCM_Resistor_SMD_AKL:R_0603_1608Metric, symbol PCM_Resistor_AKL:R_0603
- removed T1: PMV48XP_215, TO-236_SOT23_NEX, symbol MOSFET_PMV48XP,215_Nexperia:PMV48XP_215
- removed U3: LMV358IDGK, PCM_Package_SO_AKL:MSOP-8_3x3mm_P0.65mm, symbol PCM_Amplifier_Operational_AKL:LMV358IDGK
- removed UP1: LD1117S50CTR, LDO_LD1117S50CTR_STMicroelectronics:SOT-223_STM, symbol LDO_LD1117S50CTR_STMicroelectronics:LD1117S50CTR
- removed UP2: LP2985-3.3, Package_TO_SOT_SMD:SOT-23-5, symbol Regulator_Linear:LP2985-3.3
- added C1: 100nF_0603_16V, PCM_4ms_Capacitor:C_0603, symbol PCM_4ms_Capacitor:100nF_0603_16V
- added Cp1, Cp2, Cp3: 10uF_25V, Capacitor_THT:CP_Radial_D5.0mm_P2.00mm, symbol PCM_SL_Capacitors:10uF_25V
- added L1, L2: MPZ1608S101ATAH0, FerriteBead_MPZ1608S101ATAH0_TDK:IND_1608_TDK, symbol FerriteBead_MPZ1608S101ATAH0_TDK:MPZ1608S101ATAH0
- added ON2: LED_0805_Green, PCM_LED_SMD_AKL:LED_0805_2012Metric, symbol PCM_LED_AKL:LED_0805_Green
- added RON2: 1K_0603, PCM_Resistor_SMD_AKL:R_0603_1608Metric, symbol PCM_Resistor_AKL:R_0603
- added UP1: LM7805MP, PCM_Package_TO_SOT_SMD_AKL:SOT-223-3_TabPin2, symbol PCM_Voltage_Regulator_AKL:LM7805MP
- added UP2: AMS1117-3.3, Package_TO_SOT_SMD:SOT-223-3_TabPin2, symbol Regulator_Linear:AMS1117-3.3
- renumbered RN35 to RON1
Connections:
- net +5V: now also Cp2.1, UP1.3 (OUT), UP2.3 (VI); no longer C3.1
- net GND: now also C1.2, Cp1.2, Cp2.2, Cp3.2, ON2.1 (K), UP1.2, UP2.1 (GND)
- net VIN: now also Cp1.1, UP1.1 (IN); no longer C2.1
- net +3V3_2 renamed +3V3C
- new net: C3.1, Cp3.1, L1.1, L2.1, RON2.2, UP2.2 (VO)
- new net: ON2.2 (A), RON2.1
- new net +3V3A: C1.1, L1.2
- new net +3V3B: C2.1, L2.2
- no-connect marks 1 -> 0
Other:
- moved on the sheet: ON1, RON1

Commit message: Update fix schematics
Parts:
- added ON3: LED_0805_Green, PCM_LED_SMD_AKL:LED_0805_2012Metric, symbol PCM_LED_AKL:LED_0805_Green
- added RON3: 1K_0603, PCM_Resistor_SMD_AKL:R_0603_1608Metric, symbol PCM_Resistor_AKL:R_0603
Connections:
- net +3V3C: now also RON3.2
- net GND: now also ON3.1 (K)
- new net: ON3.2 (A), RON3.1
Other:
- moved on the sheet: C4, C5, C6
