File: Arduino_Shield_PoE-Wifi/PowerOverEthernet.kicad_sch (KiCad schematic)
At the start: 47 parts, among them U1 W5500, X2 25MHz 18pF

Commit message: Update
Parts:
- renumbered C1 to C7, C10 to C8
Connections:
- net +3V3D renamed +3V3B
- net GND renamed GNDB
- net GNDB: no longer C16.1, C19.1, C20.2, C21.2, C24.2, C25.2, C28.2, C29.2, C30.2, C7.1, C8.1, RJ45.10 (V-)
- new net GNDA: C16.1, C19.1, C20.2, C21.2, C24.2, C25.2, C28.2, C29.2, C30.2, C7.1, C8.1
- new net GNDPWR: RJ45.10 (V-)
Other:
- moved on the sheet: C16, R25

Commit message: Update fix schematics
Parts:
- added L_DUP1, L_SPD1: LED_0805_RED, PCM_LED_SMD_AKL:LED_0805_2012Metric, symbol PCM_LED_AKL:LED_0805_Green
- added R_DUP1, R_SPD1: 1K_0603, PCM_Resistor_SMD_AKL:R_0603_1608Metric, symbol PCM_Resistor_AKL:R_0603
Connections:
- net DUP_LED: now also R_DUP1.2
- net GNDB: now also L_DUP1.1 (K), L_SPD1.1 (K)
- net SPD_LED: now also R_SPD1.2
- new net: L_SPD1.2 (A), R_SPD1.1
- new net: L_DUP1.2 (A), R_DUP1.1

Commit message: Update Done Shield PoE
Connections:
- net +3V3B: now also RJ45.12, RJ45.14; no longer RJ45.11, RJ45.13
- net at R8.2: now also RJ45.11; no longer RJ45.12
- net at R9.2: now also RJ45.13; no longer RJ45.14
Changed lines of the file:
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@@
 			)
 		)
-		(property "Description" ""
+		(property "Description" "RJ45 PoE 10/100 Base-TX Jack with Magnetic Module"
 			(at 322.58 166.37 0)
 			(effects
@@
 					(size 1.27 1.27)
 				)
+				(hide yes)
 			)
 		)
